File: NODEMCU/Water Level Monitor and Control/Water Level Monitor and Control.kicad_pcb (KiCad board)
At the start: 2 copper layers, 130.3 x 85.6 mm, 79 parts, among them J1 12VAC_IN, J2 PUMP, K1 10A RELAY, U1 ESP8266 NODEMCU, U2 HC-SR04, U3 LM2596S-5V, U4 PCA9555D

Commit message: update from work
Parts:
- moved D10 6.62 mm to (117.3, 115.0)
- moved D12 6.62 mm to (117.3, 128.1)
- moved D8 6.62 mm to (117.2, 101.8)
- moved D9 6.62 mm to (117.2, 108.4)
- moved D3 6.62 mm to (119.8, 62.6)
- moved D11 6.62 mm to (117.3, 121.6)
- moved D13 6.62 mm to (119.8, 95.3)
- moved D15 6.62 mm to (119.8, 88.8)
- moved D16 6.62 mm to (119.8, 82.2)
- moved D4 6.62 mm to (119.8, 69.1)
- moved D7 6.62 mm to (119.8, 75.7)
- moved 5V 6.62 mm to (100.4, 138.6)
- moved 5V 6.62 mm to (122.6, 138.6)
- moved 5V 6.62 mm to (109.9, 138.6)
- moved 5V 6.62 mm to (103.6, 138.6)
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Other:
- board size 130.3 x 85.6 mm -> 123.8 x 85.6 mm
