File: NODEMCU/Water Level Monitor and Control/Water Level Monitor and Control.kicad_pcb (KiCad board)
At the start: 2 copper layers, 144.2 x 88.7 mm, 79 parts, among them J1 12VAC_IN, J2 PUMP, K1 10A RELAY, U1 ESP8266 NODEMCU, U2 HC-SR04, U3 LM2596S-5V, U4 PCA9555D

Commit message: sync updates
Parts:
- moved 5V 12.9 mm to (124.7, 141.5)
- moved 5V 12.9 mm to (127.9, 141.5)
- moved 5V 12.9 mm to (118.4, 141.5)
- moved 5V 12.9 mm to (137.3, 141.5)
- moved D8 12.9 mm to (119.4, 104.8)
- moved 5V 12.9 mm to (102.6, 141.5)
- moved 5V 12.9 mm to (112.1, 141.5)
- moved 5V 12.9 mm to (108.9, 141.5)
- moved 5V 12.9 mm to (105.8, 141.5)
- moved 5V 12.9 mm to (121.6, 141.5)
- moved 5V 12.9 mm to (134.6, 141.5)
- moved 5V 12.9 mm to (131.1, 141.5)
- moved 5V 12.9 mm to (115.3, 141.5)
- moved D10 12.9 mm to (119.4, 117.9)
- moved D11 12.9 mm to (119.5, 124.6)
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Other:
- board size 144.2 x 88.7 mm -> 131.3 x 88.7 mm

Commit message: deleted some files to fix an issue with backup file
Routing:
- net GND: track 14.1 -> 179.3 mm, vias 10 -> 12
- net +5V: track 352.6 -> 346.8 mm
- net Net-(D17-A): track 27.5 -> 23.3 mm
- net VIN: track 162.9 -> 165.7 mm
- net Net-(OC1-Pad1): track 59.9 -> 62.6 mm
- net /SCL: track 43.8 -> 41.7 mm
- net /ECHO: track 49.4 -> 51.2 mm
- net Net-(U4-~{INT}): track 18.9 -> 19.9 mm
- net Net-(D14-K): track 19.3 -> 20.2 mm
- net /PUMP_ON/OFF: track 39.3 -> 40.1 mm
- net /SDA: track 45.1 -> 44.5 mm
- net Net-(D4-A): track 178.5 -> 179.1 mm
- added copper zone on B.Cu, net (none)
- added copper zone on F.Cu, net (none)
Other:
- board text added: "K"
