File: ESP32/Dual Axis Solar Tracker/hardware/Dual Axis Solar Tracker.kicad_pcb (KiCad board)
At the start: 2 copper layers, 71 parts, among them J1 12VAC, J2 12VAC, J3 SIGNAL, J4 MOTOR, J5 12V_IN, J6 USB_C Conn, Q1 UMH3N, SW2 RESET, SW3 FLASH, U1 LM2596S-3.3V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

Commit message: Netlist class set
Parts:
- added J7: USB_C Conn, Connector_PinHeader_2.54mm:PinHeader_1x04_P2.54mm_Vertical, F.Cu at (103.7, 86.8)
- added M1: Geared Motor, TerminalBlock_4Ucon:TerminalBlock_4Ucon_1x02_P3.50mm_Vertical, F.Cu at (50.2, 67.7)
- added M2: Geared Motor, TerminalBlock_4Ucon:TerminalBlock_4Ucon_1x02_P3.50mm_Vertical, F.Cu at (60.2, 67.7)
- C10: footprint Capacitor_SMD:CP_Elec_10x12.5 -> Capacitor_SMD:CP_Elec_6.3x7.7
- J1, J2: footprint PCM_SparkFun-Connector:ScrewTerminal_1x02_P3.5mm_Horizontal_Black -> TerminalBlock_4Ucon:TerminalBlock_4Ucon_1x02_P3.50mm_Vertical
- J3: value SIGNAL -> MOTOR; footprint Connector_PinHeader_2.54mm:PinHeader_1x06_P2.54mm_Vertical -> TerminalBlock_4Ucon:TerminalBlock_4Ucon_1x02_P3.50mm_Vertical
- J4: value MOTOR -> SIGNAL; footprint PCM_SparkFun-Connector:ScrewTerminal_1x04_P3.5mm_Locking -> Connector_PinHeader_2.54mm:PinHeader_1x06_P2.54mm_Vertical
- J5: value 12V_IN -> MOTOR; footprint PCM_SparkFun-Connector:ScrewTerminal_1x02_P3.5mm_Horizontal_Black -> TerminalBlock_4Ucon:TerminalBlock_4Ucon_1x02_P3.50mm_Vertical
- J6: value USB_C Conn -> 12V_IN; footprint Connector_PinHeader_2.54mm:PinHeader_1x04_P2.54mm_Vertical -> TerminalBlock_4Ucon:TerminalBlock_4Ucon_1x02_P3.50mm_Vertical
- R11, R13, R15, R5, R7: footprint OptoDevice:R_LDR_5.1x4.3mm_P3.4mm_Vertical -> Connector_PinHeader_2.54mm:PinHeader_1x02_P2.54mm_Vertical
- moved J6 115.4 mm to (40.1, 67.7)
- moved C15 100.4 mm to (45.6, 113.0)
- moved J3 99.8 mm to (60.2, 57.1)
- moved J1 85.4 mm to (40.1, 57.1)
- moved J2 84.5 mm to (50.2, 57.1)
- moved Y1 76.3 mm to (81.2, 67.5)
- moved J5 73.8 mm to (70.3, 57.1)
- moved C11 68.4 mm to (58.6, 96.4)
- moved C12 68.4 mm to (58.6, 99.4)
- moved C14 68.4 mm to (58.6, 102.4)
- moved C16 68.4 mm to (58.6, 105.4)
- moved C17 68.4 mm to (58.6, 108.4)
- moved C19 68.4 mm to (58.6, 111.4)
- moved C20 68.4 mm to (63.4, 96.4)
- moved C21 68.4 mm to (63.4, 99.4)
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Connections:
- D3 pad 2: Net-(D3-Pad2) -> Net-(J1-Pin_2)
- D3 pad 3: Net-(D3-Pad3) -> Net-(J1-Pin_1)
- D4 pad 2: Net-(D4-Pad2) -> Net-(J2-Pin_2)
- D4 pad 3: Net-(D4-Pad3) -> Net-(J2-Pin_1)
- J3 pad 1: /GPIO14 -> Net-(J3-Pin_1)
- J3 pad 2: /GPIO27 -> Net-(J3-Pin_2)
- J4 pad 1: Net-(J4-Pin_1) -> /GPIO14
- J4 pad 2: Net-(J4-Pin_2) -> /GPIO27
- J4 pad 3: Net-(J4-Pin_3) -> /GPIO26
- J4 pad 4: Net-(J4-Pin_4) -> /GPIO33
- J5 pad 1: +12V -> Net-(J5-Pin_1)
- J5 pad 2: GND -> Net-(J5-Pin_2)
- J6 pad 1: GND -> +12V
- J6 pad 2: Net-(J6-Pin_2) -> GND
- U4 pad 5: Net-(J6-Pin_2) -> /+
- U4 pad 6: Net-(J6-Pin_3) -> /-

Commit message: Ready for Production
Parts:
- added  : LOGO, logo:CULogo, B.Cu at (182.1, 93.1)
- added M2: MountingHole_2.2mm_M2_Pad, MountingHole:MountingHole_2.2mm_M2_Pad, F.Cu at (190.1, 118.6)
- added M2: MountingHole_2.2mm_M2_Pad, MountingHole:MountingHole_2.2mm_M2_Pad, F.Cu at (97.8, 120.1)
- added M2: MountingHole_2.2mm_M2_Pad, MountingHole:MountingHole_2.2mm_M2_Pad, F.Cu at (97.8, 49.5)
- added M2: MountingHole_2.2mm_M2_Pad, MountingHole:MountingHole_2.2mm_M2_Pad, F.Cu at (192.6, 49.5)
- added SW1: RotaryEncoder, Connector_PinHeader_2.54mm:PinHeader_1x06_P2.54mm_Vertical, F.Cu at (181.6, 69.3)
- D8: footprint Diode_THT:D_DO-41_SOD81_P10.16mm_Horizontal -> Diode_SMD:D_SMA
- J1, J2, J3, J5, J6, M1, M2: footprint TerminalBlock_4Ucon:TerminalBlock_4Ucon_1x02_P3.50mm_Vertical -> TerminalBlock_Phoenix:TerminalBlock_Phoenix_PT-1,5-2-3.5-H_1x02_P3.50mm_Horizontal
- moved C18 133.7 mm to (166.2, 71.9)
- moved C15 128.1 mm to (162.4, 60.5), turned to 180 degrees
- moved C13 123.9 mm to (155.4, 66.8), turned to 180 degrees
- moved D8 123.7 mm to (167.2, 66.8)
- moved D1 123.0 mm to (193.0, 57.2), turned to 90 degrees
- moved D2 122.7 mm to (192.8, 63.5), turned to 90 degrees
- moved D5 122.4 mm to (192.7, 69.9), turned to 90 degrees
- moved D6 122.1 mm to (192.7, 76.5), turned to 90 degrees
- moved J6 115.6 mm to (154.0, 87.5), turned to -90 degrees
- moved C17 110.7 mm to (161.0, 66.3)
- moved J5 110.5 mm to (162.5, 117.9)
- moved R4 109.6 mm to (188.3, 73.8)
- moved R3 109.4 mm to (188.4, 67.2)
- moved R2 109.3 mm to (188.4, 60.8)
- moved R1 109.3 mm to (188.5, 54.5)
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Connections:
- D3 pad 2: Net-(J1-Pin_2) -> Net-(J1-Pin_1)
- D3 pad 3: Net-(J1-Pin_1) -> Net-(J1-Pin_2)
- D4 pad 2: Net-(J2-Pin_2) -> Net-(J2-Pin_1)
- D4 pad 3: Net-(J2-Pin_1) -> Net-(J2-Pin_2)
- M2 pad 1: Net-(J5-Pin_2) -> Net-(J5-Pin_1)
- M2 pad 2: Net-(J5-Pin_1) -> Net-(J5-Pin_2)
Routing:
- net +3.3V: track 0.00 -> 260.7 mm, vias 0 -> 7
- net Net-(J3-Pin_2): track 0.00 -> 96.6 mm
- net /GPIO19: track 0.00 -> 90.2 mm
- net /GPIO17: track 0.00 -> 87.5 mm, vias 0 -> 2
- net /GPIO5: track 0.00 -> 80.4 mm, vias 0 -> 2
- net /GPIO27: track 0.00 -> 66.5 mm, vias 0 -> 6
- net Net-(J3-Pin_1): track 0.00 -> 66.2 mm
- net VCC: track 0.00 -> 65.5 mm, vias 0 -> 13
- net +12V: track 0.00 -> 65.2 mm
- net /GPIO14: track 0.00 -> 65.1 mm, vias 0 -> 2
- net /GPIO33: track 0.00 -> 63.2 mm, vias 0 -> 2
- net /GPIO15: track 0.00 -> 63.0 mm, vias 0 -> 2
- net /GPIO32: track 0.00 -> 62.9 mm, vias 0 -> 2
- net /GPIO23: track 0.00 -> 62.5 mm
- net /GPIO25: track 0.00 -> 61.9 mm, vias 0 -> 2
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- added copper zone on B.Cu, net +12V
- added copper zone on B.Cu, net GND
- added copper zone on F.Cu, net GND
- added copper zone on B.Cu, net VCC
- added copper zone on F.Cu, net VCC
Other:
- board outline added: 101.2 x 76.6 mm
- board text added: "+12V"
- board text added: "12VAC"
- board text added: "A"
- board text added: "AZIMUTH"
- board text added: "B"
- board text added: "ELEVATION"
- board text added: "ENA"
- board text added: "ENB"
- board text added: "ENCODER"
- board text added: "GND"
- board text added: "IN1"
- board text added: "IN2"
- board text added: "IN3"
- board text added: "IN4"
- board text added: "LDR's"
- board text added: "MICROCONTROLLER"
- board text added: "MOTOR DRIVER"
- board text added: "SW"

Commit message: UPDATE FROM WORK
Parts:
- moved C15 0.67 mm to (162.4, 61.1)
Other:
- board text added: "+5V"
- board text added: "D+"
- board text added: "D-"
- board text added: "USB"
Changed lines of the file:
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@@
 	(footprint "Capacitor_THT:CP_Radial_D5.0mm_P2.00mm"
 		(layer "F.Cu")
-		(at 162.42 60.47 180)
+		(at 162.415 61.14 180)
 		(descr "CP, Radial series, Radial, pin pitch=2.00mm, diameter=5mm, height=7mm, Electrolytic Capacitor")
 		(tags "CP Radial series Radial pin pitch 2.00mm diameter 5mm height 7mm Electrolytic Capacitor")
@@
 			(at 2.485 4.705 0)
 			(layer "F.SilkS")
+			(hide yes)
 			(effects
 				(font
@@
 		)
 	)
+	(gr_text "USB"
+		(at 156.295 52.57 0)
+		(layer "F.SilkS")
+		(effects
+			(font
+				(size 1.5 1.5)
+				(thickness 0.3)
+				(bold yes)
+			)
+			(justify left bottom)
+		)
+	)
 	(gr_text "ELEVATION"
 		(at 137.875 113.045 0)
@@
 		)
 	)
+	(gr_text "GND"
+		(at 155.76 55.305 90)
+		(layer "B.SilkS")
+		(effects
+			(font
+				(size 1.5 1.5)
+				(thickness 0.3)
+				(bold yes)
+			)
+			(justify left bottom mirror)
+		)
+	)
+	(gr_text "D-"
+		(at 160.835 55.305 90)
+		(layer "B.SilkS")
+		(effects
+			(font
+				(size 1.5 1.5)
+				(thickness 0.3)
+				(bold yes)
+			)
+			(justify left bottom mirror)
+		)
+	)
 	(gr_text "ENA"
 		(at 158.255 103.176 0)
@@
 		)
 	)
+	(gr_text "D+"
+		(at 158.285 55.305 90)
+		(layer "B.SilkS")
+		(effects
+			(font
+				(size 1.5 1.5)
+				(thickness 0.3)
+				(bold yes)
+			)
+			(justify left bottom mirror)
+		)
+	)
 	(gr_text "B"
 		(at 184.585 65.255 0)
@@
 		)
 	)
+	(gr_text "+5V"
+		(at 163.45 55.305 90)
+		(layer "B.SilkS")
+		(effects
+			(font
+				(size 1.5 1.5)
+				(thickness 0.3)
+				(bold yes)
+			)
+			(justify left bottom mirror)
+		)
+	)
 	(via
 		(at 181.375 106.55)
@@
 	)
 	(segment
-		(start 162.0275 64.6625)
-		(end 162.42 64.27)
+		(start 157.0775 70.8775)
+		(end 157.66 71.46)
+		(width 0.8)
+		(layer "F.Cu")
+		(net 10)
+	)
+	(segment
+		(start 162.42 61.145)
+		(end 162.415 61.14)
 		(width 0.8)
 		(layer "F.Cu")
@@
 	(segment
 		(start 162.42 64.27)
-		(end 162.42 60.47)
+		(end 162.42 61.145)
 		(width 0.8)
 		(layer "F.Cu")
@@
 	)
 	(segment
-		(start 157.0775 70.8775)
-		(end 157.66 71.46)
+		(start 162.0275 64.6625)
+		(end 162.42 64.27)
 		(width 0.8)
 		(layer "F.Cu")
@@
 	)
 	(segment
+		(start 162.42 61.135)
+		(end 162.415 61.14)
+		(width 0.8)
+		(layer "B.Cu")
+		(net 10)
+	)
+	(segment
 		(start 162.42 54.39)
-		(end 162.42 60.47)
+		(end 162.42 61.135)
 		(width 0.8)
 		(layer "B.Cu")
