File: ESP32/Solar Powered Irrigation System/hardware/Solar Powered Irrigation System.kicad_sch (KiCad schematic)
At the start: 0 parts

Commit message: Done with Schematic Diagram
Parts:
- added BT1: Battery_Cell, symbol Device:Battery_Cell
- added BZ1: Buzzer, Buzzer_Beeper:Buzzer_15x7.5RM7.6, symbol Device:Buzzer
- added C1, C10, C18, C2, C21, C22, C3, C4, C5, C6: 100nF, Capacitor_SMD:C_0805_2012Metric_Pad1.18x1.45mm_HandSolder, symbol PCM_SL_Capacitors:104_Ceramic
- added C11, C17: 100nF, Capacitor_SMD:C_0805_2012Metric_Pad1.18x1.45mm_HandSolder, symbol Device:C_Small
- added C12, C7: 4.7uF/16V, Capacitor_Tantalum_SMD:CP_EIA-3528-21_Kemet-B_HandSolder, symbol PCM_SL_Capacitors:4.7uF_16V
- added C13, C14: 680uF_35V, Capacitor_SMD:CP_Elec_10x12.5, symbol PCM_SL_Capacitors:470uF_35V
- added C15, C16: 22pF, Capacitor_SMD:C_0805_2012Metric_Pad1.18x1.45mm_HandSolder, symbol Device:C_Small
- added C19, C20: 220uF_16V, Capacitor_SMD:CP_Elec_6.3x7.7, symbol PCM_SL_Capacitors:470uF_35V
- added C8: 10uF_16V, Capacitor_THT:CP_Radial_D5.0mm_P2.00mm, symbol PCM_SL_Capacitors:10uF_16V
- added C9: 470nF, Capacitor_SMD:C_0805_2012Metric_Pad1.18x1.45mm_HandSolder, symbol PCM_SL_Capacitors:104_Ceramic
- added D1: 3.3V, Diode_SMD:D_SOD-123, symbol Device:D_Zener_Small
- added D2: 1N5819, Diode_THT:D_DO-41_SOD81_P10.16mm_Horizontal, symbol Diode:1N5819
- added D3, D5: Red, LED_THT:LED_D3.0mm, symbol SparkFun-LED:LED_Red_0603
- added D4: 1N5819, Diode_SMD:D_SMA, symbol Diode:1N5819
- added D6: Green, LED_THT:LED_D3.0mm, symbol SparkFun-LED:LED_Red_0603
- added D7, D8: 1N5824, Diode_SMD:D_SMA, symbol Diode:1N5822
- added J1, J5: GAS SENSOR, Connector_PinSocket_2.54mm:PinSocket_1x04_P2.54mm_Vertical, symbol Connector:Screw_Terminal_01x04
- added J10: -BATT, symbol Connector:Screw_Terminal_01x01
- added J11: +BATT, symbol Connector:Screw_Terminal_01x01
- added J12: +5V, TestPoint:TestPoint_Keystone_5015_Micro_Mini, symbol Connector:Screw_Terminal_01x01
- added J13: -5V, TestPoint:TestPoint_Keystone_5015_Micro_Mini, symbol Connector:Screw_Terminal_01x01
- added J2: SOIL SENSOR, Connector_PinHeader_2.54mm:PinHeader_1x03_P2.54mm_Vertical, symbol Connector:Screw_Terminal_01x03
- added J3: AM2301A, Connector_PinHeader_2.54mm:PinHeader_1x03_P2.54mm_Vertical, symbol Connector:Screw_Terminal_01x03
- added J4: OLED SCREEN, Connector_PinSocket_2.54mm:PinSocket_1x04_P2.54mm_Vertical, symbol Connector:Screw_Terminal_01x04
- added J6: SOLAR IN, symbol Connector_Generic:Conn_01x02
- added J7: USB_C Conn, Connector_PinHeader_2.54mm:PinHeader_1x04_P2.54mm_Vertical, symbol Connector:Screw_Terminal_01x04
- added J8: +IN, TestPoint:TestPoint_Keystone_5015_Micro_Mini, symbol Connector:Screw_Terminal_01x01
- added J9: -IN, TestPoint:TestPoint_Keystone_5015_Micro_Mini, symbol Connector:Screw_Terminal_01x01
- added JP1: ~, Jumper:SolderJumper-2_P1.3mm_Open_Pad1.0x1.5mm, symbol SparkFun-Jumper:SolderJumper_2_Open
- added L1, L2: 33uH, Inductor_SMD:L_12x12mm_H6mm, symbol Device:L_Small
- added OC1: PC817XI, PCM_Package_DIP_AKL:SMDIP-4_W9.53mm, symbol PCM_Optocoupler_AKL:PC817XI
- added Q1, Q2: IRLML6344, PCM_Package_TO_SOT_SMD_AKL:SOT-23, symbol PCM_Transistor_MOSFET_AKL:IRLML6344
- added Q3: UMH3N, Package_TO_SOT_SMD:SOT-363_SC-70-6, symbol Transistor_BJT:UMH3N
- added R1, R11, R2, R3, R4, R5, R9: 10k, Resistor_SMD:R_0805_2012Metric, symbol PCM_SL_Resistors:10k
- added R10, R12, R13: 330R, Resistor_SMD:R_0805_2012Metric, symbol PCM_SL_Resistors:1M
- added R6: 20k, Resistor_SMD:R_0805_2012Metric, symbol PCM_SL_Resistors:10k
- added R7: 1k, Resistor_SMD:R_0805_2012Metric, symbol PCM_SL_Resistors:10k
- added R8: 2k, Resistor_SMD:R_0805_2012Metric, symbol PCM_SL_Resistors:10k
- added SW1: RotaryEncoder, symbol Device:RotaryEncoder_Switch_MP
- added SW2: RESET, Button_Switch_SMD:SW_SPST_CK_KXT3, symbol PCM_SL_Devices:Push_Button
- added SW3: FLASH, Button_Switch_SMD:SW_SPST_CK_KXT3, symbol PCM_SL_Devices:Push_Button
- added U1: AMS1117-3.3, Package_TO_SOT_SMD:SOT-223-3_TabPin2, symbol Regulator_Linear:AMS1117-3.3
- added U2: ESP32-WROOM, RF_Module:ESP32-WROOM-32U, symbol SparkFun-RF:ESP32-WROOM
- added U3, U4: LM2596S-3.3V, Package_TO_SOT_SMD:TO-263-5_TabPin6, symbol Regulator_Switching:LM2596S-3.3
- added U5: CH340C, Package_SO:SOIC-16_3.9x9.9mm_P1.27mm, symbol Interface_USB:CH340C
- added Y1: 12MHz, Crystal:Crystal_HC49-4H_Vertical, symbol PCM_SL_Devices:Crystal_16MHz
Connections:
- new net: D5.2 (A), R12.2
- new net: C11.2, C7.1, C8.1, D2.1 (K), J7.4 (Pin_4), U1.3 (VI)
- new net: D7.1 (K), L1.1, U3.2 (OUT)
- new net: OC1.1, R4.2
- new net: J7.2 (Pin_2), U5.5 (UD+)
- new net: J7.3 (Pin_3), U5.6 (UD-)
- new net: D3.2 (A), R10.2
- new net: C12.1, D4.2 (A), U1.2 (VO)
- new net: BT1.2 (-), J10.1 (Pin_1)
- new net: D6.2 (A), R13.2
- new net: J5.3 (Pin_3), R7.1
- new net: J1.2 (Pin_2), Q2.3 (D)
- new net: J1.4 (Pin_4), Q1.3 (D)
- new net: D8.1 (K), L2.1, U4.2 (OUT)
- new net: C17.2, JP1.1 (A), U5.4 (V3)
- new net: C15.1, U5.7 (Xi), Y1.2
- new net: C16.1, U5.8 (Xo), Y1.1
- new net: J6.2 (Pin_2), J9.1 (Pin_1)
- new net: J6.1 (Pin_1), J8.1 (Pin_1)
- new net: BZ1.2 (-), OC1.4
- new net: BT1.1 (+), J11.1 (Pin_1)
- new net +3.3V: C1.2, C10.2, C18.1, C19.1, C2.1, C21.2, C3.2, D4.1 (K), J2.2 (Pin_2), J3.3 (Pin_3), J4.3 (Pin_3), JP1.2 (B), L1.2, R1.1, R11.2, R12.1, R13.1, R2.2, R3.1, R9.2, U2.2 (VDD), U3.4 (FB), U5.16 (VCC)
- new net +5V: BZ1.1 (+), C20.1, C22.2, C6.2, J1.1 (Pin_1), J1.3 (Pin_3), J5.1 (Pin_1), L2.2, U4.4 (FB)
- new net +BATT: R5.1
- new net DTR: Q3.2 (B1), Q3.4 (E2), U5.13 (~{DTR})
- new net EN: C9.2, Q3.6 (C1), R9.1, SW2.2, U2.3 (EN)
- new net GND: C1.1, C10.1, C11.1, C12.2, C13.2, C14.2, C15.2, C16.2, C17.1, C18.2, C19.2, C2.2, C20.2, C21.1, C22.1, C3.1, C4.1, C5.1, C6.1, C7.2, C8.2, C9.1, D1.2 (A), D2.2 (A), D3.1 (K), D7.2 (A), D8.2 (A), J13.1 (Pin_1), J2.1 (Pin_1), J3.1 (Pin_1), J4.4 (Pin_4), J5.4 (Pin_4), J7.1 (Pin_1), OC1.2, OC1.3, Q1.2 (S), Q2.2 (S), R6.1, R8.1, SW1.C, SW1.MP, SW1.S2, SW2.1, SW3.1, U1.1 (GND), U2.1 (GND), U2.15 (GND), U2.38 (GND), U2.39 (GND), U3.3 (GND), U3.5 (~{ON}/OFF), U3.6 (GND), U4.3 (GND), U4.5 (~{ON}/OFF), U4.6 (GND), U5.1 (GND)
- new net GPIO0: Q3.3 (C2), R11.1, SW3.2, U2.25 (IOA0)
- new net GPIO12: R7.2, R8.2, U2.14 (IOA12)
- new net GPIO13: U2.16 (IOA13)
- new net GPIO14: J5.2 (Pin_2), U2.13 (IOA14)
- new net GPIO15: U2.23 (IOA15)
- new net GPIO16: Q1.1 (G), U2.27 (IO16)
- new net GPIO17: U2.28 (IO17)
- new net GPIO18/SCK: U2.30 (IO18)
- new net GPIO19/MISO: U2.31 (IO19)
- new net GPIO1/TX: D5.1 (K), U2.35 (TXD0/IO1), U5.3 (RXD)
- new net GPIO2: R10.1, U2.24 (IOA2)
- new net GPIO23/MOSI: U2.37 (IO23)
- new net GPIO25: R3.2, SW1.A, U2.10 (IOA25)
- new net GPIO26: R2.1, SW1.B, U2.11 (IOA26)
- new net GPIO27: SW1.S1, U2.12 (IOA27)
- new net GPIO32: C4.2, J3.2 (Pin_2), R1.2, U2.8 (IOA32)
- new net GPIO33: Q2.1 (G), U2.9 (IOA33)
- new net GPIO34: J2.3 (Pin_3), U2.6 (IA34)
- new net GPIO35: C5.2, D1.1 (K), R5.2, R6.2, U2.7 (IA35)
- new net GPIO36: U2.4 (IA36)
- new net GPIO39: U2.5 (IA39)
- new net GPIO3/RX: D6.1 (K), U2.34 (RXD0/IO3), U5.2 (TXD)
- new net GPIO4: R4.1, U2.26 (IOA4)
- new net GPIO5/CS: U2.29 (IO5)
- new net RTS: Q3.1 (E1), Q3.5 (B2), U5.14 (~{RTS})
- new net SCL: J4.2 (Pin_2), U2.36 (IO22)
- new net SDA: J4.1 (Pin_1), U2.33 (IO21)
- new net VCC: C13.1, C14.1, J12.1 (Pin_1), U3.1 (VIN), U4.1 (VIN)
- no-connect marks 0 -> 9
Other:
- note added: "BATTERY LEVEL"
- note added: "BUZZER"
- note added: "CHARGE/DISCHARGE"
- note added: "CONTROL & COMMAND"
- note added: "DEBUGGING & PROGRAMMING"
- note added: "If CH340G is used"
- note added: "MODULE"
- note added: "MONITORING SCREEN"
- note added: "OLED DISPLAY"
- note added: "POWER SUPPLY"
- note added: "PUMP SYSTEM"
- note added: "SOIL SENSOR"
- note added: "TEMPERATURE & HUMIDITY SENSOR"
- note added: "ULTRASONIC SENSOR"
- note added: "USER INPUT"

Commit message: Update from home
Parts:
- added J11: INPUT, TerminalBlock_Phoenix:TerminalBlock_Phoenix_PT-1,5-2-3.5-H_1x02_P3.50mm_Horizontal, symbol Connector_Generic:Conn_01x02
- added J15: BSEN, TestPoint:TestPoint_Keystone_5015_Micro_Mini, symbol Connector:Screw_Terminal_01x01
- added R14, R15: 10k, Resistor_SMD:R_0805_2012Metric, symbol PCM_SL_Resistors:10k
- D2: footprint Diode_THT:D_DO-41_SOD81_P10.16mm_Horizontal -> Diode_SMD:D_SMA
- J1: value GAS SENSOR -> PUMP; footprint Connector_PinSocket_2.54mm:PinSocket_1x04_P2.54mm_Vertical -> TerminalBlock_Phoenix:TerminalBlock_Phoenix_PT-1,5-4-3.5-H_1x04_P3.50mm_Horizontal
- J13: renamed from J12; now left out of the parts list
- J14: renamed from J13; now left out of the parts list
- J5: value GAS SENSOR -> Ultra Sonic
- OC1: footprint PCM_Package_DIP_AKL:SMDIP-4_W9.53mm -> Package_DIP:DIP-4_W7.62mm_SMDSocket_SmallPads
- Q1, Q2: footprint PCM_Package_TO_SOT_SMD_AKL:SOT-23 -> Package_TO_SOT_SMD:SOT-23_Handsoldering
- SW1: footprint (none) -> Connector_PinHeader_2.54mm:PinHeader_1x06_P2.54mm_Vertical
- renumbered J11 to J12
Connections:
- net +3.3V: now also R14.1, R15.1
- net +BATT: now also J15.1 (Pin_1)
- net GND: now also SW1.2 (C), SW1.5 (S2), SW1.6 (MP), J11.2 (Pin_2); no longer SW1.C, SW1.MP, SW1.S2
- net GPIO25: now also SW1.1 (A); no longer SW1.A
- net GPIO26: now also SW1.3 (B); no longer SW1.B
- net GPIO27: now also SW1.4 (S1); no longer SW1.S1
- net SCL: now also R15.2
- net SDA: now also R14.2
- net VCC: now also J11.1 (Pin_1)
- net +: now reaches J7.2 (Pin_2), U5.5 (UD+)
- net -: now reaches J7.3 (Pin_3), U5.6 (UD-)
