File: ESP32/Smart Posture Corrector/hardware/Smart Posture Corrector.kicad_pcb (KiCad board)
At the start: 2 copper layers, 106.5 x 93.9 mm, 64 parts, among them J1 MPU6050, J10 -5V, J11 USB_C Conn, J15 SD MODULE, J24 BSENS, J5 +IN, J6 -IN, J9 +5V, M1 Motor_DC, Q1 UMH3N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

Commit message: Update from home
Parts:
- moved C1 5.81 mm to (139.0, 122.7), turned to 180 degrees
- moved D2 3.26 mm to (136.4, 133.9)
- moved C13 3.26 mm to (128.9, 133.7)
- moved C10 2.93 mm to (131.4, 126.0)
- moved C3 2.91 mm to (145.5, 141.8)
- moved L1 2.82 mm to (153.2, 127.3)
- moved C8 2.27 mm to (131.1, 82.0), turned to 90 degrees
- moved U1 1.88 mm to (166.3, 142.5)
- moved M1 1.48 mm to (167.4, 117.9)
- moved C6 1.42 mm to (130.6, 76.0)
Connections:
- M1 pad 1: VCC -> +3.3V
Routing:
- net Net-(M1--): vias 0 -> 1
- net GND: vias 0 -> 2
- net +3.3V: vias 0 -> 1
Other:
- board size 106.5 x 93.9 mm -> 105.6 x 92.8 mm
- board text added: "+"
- board text added: "+5V"
- board text added: "-"
- board text added: "100%"
- board text added: "25%"
- board text added: "50%"
- board text added: "75%"
- board text added: "AD0"
- board text added: "BSEN"
- board text added: "D+"
- board text added: "D-"
- board text added: "INT"
- board text added: "MOTOR"
- board text added: "P_ON"
- board text added: "SCL"
- board text added: "SDA"
- board text added: "USB"
- board text added: "XCL"
- board text added: "XDA"
- board text removed: "BSENSE"

Commit message: ready for production
Parts:
- added G***: LOGO, logo:CULogo, B.Cu at (139.1, 129.3)
- added M2: MountingHole_2.5mm_Pad, MountingHole:MountingHole_2.5mm_Pad, F.Cu at (127.4, 147.9)
- added M2: MountingHole_2.5mm_Pad, MountingHole:MountingHole_2.5mm_Pad, F.Cu at (127.5, 61.6)
- added M2: MountingHole_2.5mm_Pad, MountingHole:MountingHole_2.5mm_Pad, F.Cu at (173.6, 147.9)
- moved U1 5.82 mm to (160.5, 142.7)
- moved C14 5.64 mm to (132.8, 65.2)
- moved C3 2.38 mm to (143.1, 141.8)
- moved OC1 2.15 mm to (163.5, 90.0)
- moved R8 1.71 mm to (170.1, 84.1)
- moved L1 1.61 mm to (151.5, 127.3)
- moved C8 1.51 mm to (131.4, 83.5)
- moved C9 1.51 mm to (133.5, 89.2)
- moved J11 1.51 mm to (126.9, 67.8)
- moved C6 1.51 mm to (130.9, 77.5)
- moved D1 1.51 mm to (126.9, 82.2)
- moved D4 1.51 mm to (134.5, 97.6)
- moved U2 1.51 mm to (128.5, 96.8)
- moved C4 1.51 mm to (127.7, 89.2)
- moved Y1 1.15 mm to (138.3, 79.3)
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Connections:
- net Net-(J11-Pin_2) renamed /+
- net Net-(J11-Pin_3) renamed /-
Routing:
- net +3.3V: track 0.00 -> 286.8 mm, vias 1 -> 4
- net /GPIO34: track 0.00 -> 94.4 mm, vias 0 -> 2
- net /CS: track 0.00 -> 78.2 mm, vias 0 -> 6
- net /MOSI: track 0.00 -> 76.7 mm, vias 0 -> 6
- net /SCL: track 0.00 -> 70.4 mm, vias 0 -> 5
- net /SCK: track 0.00 -> 69.3 mm, vias 0 -> 2
- net /MISO: track 0.00 -> 67.7 mm, vias 0 -> 2
- net /SDA: track 0.00 -> 63.3 mm, vias 0 -> 5
- net Net-(M1--): track 0.00 -> 58.9 mm, vias 1 -> 2
- net /GPIO3/RX: track 0.00 -> 58.1 mm, vias 0 -> 2
- net /GPIO2: track 0.00 -> 53.9 mm, vias 0 -> 2
- net /GPIO27: track 0.00 -> 50.5 mm, vias 0 -> 2
- net /GPIO17: track 0.00 -> 50.0 mm
- net /GPIO13: track 0.00 -> 50.0 mm
- net /GPIO0: track 0.00 -> 49.3 mm, vias 0 -> 4
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- added copper zone on B.Cu, net 5V
- added copper zone on F.Cu, net 5V
- added copper zone on B.Cu, net GND
- added copper zone on F.Cu, net GND
- added copper zone on B.Cu, net VCC
- added copper zone on F.Cu, net VCC
Other:
- board size 105.6 x 92.8 mm -> 105.6 x 92.7 mm
