File: ESP32/Smart Robotic Car With PID control/hardware/Smart Robotic Car With PID control.kicad_sch (KiCad schematic)
At the start: 0 parts

Commit message: Update from work
Parts:
- added BT1, BT2, BT3, BT4, BT5, BT6: Battery_Cell, symbol Device:Battery_Cell
- added C1, C13, C15, C2, C7: 100nF, Capacitor_SMD:C_0805_2012Metric_Pad1.18x1.45mm_HandSolder, symbol PCM_SL_Capacitors:104_Ceramic
- added C10: 220uF_16V, Capacitor_SMD:CP_Elec_6.3x7.7, symbol PCM_SL_Capacitors:470uF_35V
- added C11, C12: 22pF, Capacitor_SMD:C_0805_2012Metric_Pad1.18x1.45mm_HandSolder, symbol Device:C_Small
- added C14, C8: 100nF, Capacitor_SMD:C_0805_2012Metric_Pad1.18x1.45mm_HandSolder, symbol Device:C_Small
- added C3: 680uF_35V, Capacitor_SMD:CP_Elec_10x12.5, symbol PCM_SL_Capacitors:470uF_35V
- added C4, C9: 4.7uF/16V, Capacitor_Tantalum_SMD:CP_EIA-3528-21_Kemet-B_HandSolder, symbol PCM_SL_Capacitors:4.7uF_16V
- added C5: 470nF, Capacitor_SMD:C_0805_2012Metric_Pad1.18x1.45mm_HandSolder, symbol PCM_SL_Capacitors:104_Ceramic
- added C6: 10uF_16V, Capacitor_THT:CP_Radial_D5.0mm_P2.00mm, symbol PCM_SL_Capacitors:10uF_16V
- added D1, D4: 1N5819, Diode_SMD:D_SMA, symbol Diode:1N5819
- added D10, D3, D5, D7, D8, D9: Red, LED_THT:LED_D3.0mm, symbol SparkFun-LED:LED_Red_0603
- added D2: 1N5824, Diode_SMD:D_SMA, symbol Diode:1N5822
- added D6: Green, LED_THT:LED_D3.0mm, symbol SparkFun-LED:LED_Red_0603
- added J1: MPU6050, symbol Connector:Screw_Terminal_01x08
- added J10: -5V, TestPoint:TestPoint_Keystone_5015_Micro_Mini, symbol Connector:Screw_Terminal_01x01
- added J11: USB_C Conn, Connector_PinHeader_2.54mm:PinHeader_1x04_P2.54mm_Vertical, symbol Connector:Screw_Terminal_01x04
- added J2: Ultra Sonic, Connector_PinSocket_2.54mm:PinSocket_1x04_P2.54mm_Vertical, symbol Connector:Screw_Terminal_01x04
- added J24: BSENS, Connector_Wire:SolderWire-0.1sqmm_1x01_D0.4mm_OD1mm, symbol Connector:Screw_Terminal_01x01
- added J3: CHARGER IN, symbol Connector_Generic:Conn_01x02
- added J5: +IN, TestPoint:TestPoint_Keystone_5015_Micro_Mini, symbol Connector:Screw_Terminal_01x01
- added J6: -IN, TestPoint:TestPoint_Keystone_5015_Micro_Mini, symbol Connector:Screw_Terminal_01x01
- added J7: -BATT, symbol Connector:Screw_Terminal_01x01
- added J8: +BATT, symbol Connector:Screw_Terminal_01x01
- added J9: +5V, TestPoint:TestPoint_Keystone_5015_Micro_Mini, symbol Connector:Screw_Terminal_01x01
- added JP1: ~, Jumper:SolderJumper-2_P1.3mm_Open_Pad1.0x1.5mm, symbol SparkFun-Jumper:SolderJumper_2_Open
- added L1: 33uH, Inductor_SMD:L_12x12mm_H6mm, symbol Device:L_Small
- added Q1: UMH3N, Package_TO_SOT_SMD:SOT-363_SC-70-6, symbol Transistor_BJT:UMH3N
- added R1, R13, R14, R15, R17: 10k, Resistor_SMD:R_0805_2012Metric, symbol PCM_SL_Resistors:10k
- added R16, R18, R19, R4, R5, R6, R7: 330R, Resistor_SMD:R_0805_2012Metric, symbol PCM_SL_Resistors:1M
- added R2: 20k, Resistor_SMD:R_0805_2012Metric, symbol PCM_SL_Resistors:10k
- added R3: 1k, Resistor_SMD:R_0805_2012Metric, symbol PCM_SL_Resistors:10k
- added R8: 2k, Resistor_SMD:R_0805_2012Metric, symbol PCM_SL_Resistors:10k
- added SW2: RESET, Button_Switch_SMD:SW_SPST_CK_KXT3, symbol PCM_SL_Devices:Push_Button
- added SW3: FLASH, Button_Switch_SMD:SW_SPST_CK_KXT3, symbol PCM_SL_Devices:Push_Button
- added U1: LM2596S-3.3V, Package_TO_SOT_SMD:TO-263-5_TabPin6, symbol Regulator_Switching:LM2596S-3.3
- added U2: AMS1117-3.3, Package_TO_SOT_SMD:SOT-223-3_TabPin2, symbol Regulator_Linear:AMS1117-3.3
- added U3: ESP32-WROOM, RF_Module:ESP32-WROOM-32U, symbol SparkFun-RF:ESP32-WROOM
- added U4: CH340C, Package_SO:SOIC-16_3.9x9.9mm_P1.27mm, symbol Interface_USB:CH340C
- added Y1: 12MHz, Crystal:Crystal_HC49-4H_Vertical, symbol PCM_SL_Devices:Crystal_16MHz
Connections:
- new net: C14.2, JP1.1 (A), U4.4 (V3)
- new net: J11.2 (Pin_2), U4.5 (UD+)
- new net: J11.3 (Pin_3), U4.6 (UD-)
- new net: C11.1, U4.7 (Xi), Y1.2
- new net: C12.1, U4.8 (Xo), Y1.1
- new net: D5.2 (A), R18.2
- new net: BT1.2 (-), BT3.1 (+)
- new net: BT3.2 (-), BT4.2 (-), J7.1 (Pin_1)
- new net: D9.2 (A), R6.2
- new net: BT5.1 (+), BT6.1 (+), J8.1 (Pin_1)
- new net: BT1.1 (+), BT5.2 (-)
- new net: C9.1, D4.2 (A), U2.2 (VO)
- new net: D3.2 (A), R16.2
- new net: D8.2 (A), R5.2
- new net: D2.1 (K), L1.1, U1.2 (OUT)
- new net: J3.1 (Pin_1), J5.1 (Pin_1)
- new net: J2.3 (Pin_3), R3.1
- new net: D7.2 (A), R4.2
- new net: BT2.2 (-), BT4.1 (+)
- new net: BT2.1 (+), BT6.2 (-)
- new net: D10.2 (A), R7.2
- new net: D6.2 (A), R19.2
- new net +3.3V: C10.1, C13.2, C15.1, C7.2, D4.1 (K), J1.1 (Pin_1), JP1.2 (B), L1.2, R13.1, R14.2, R15.2, R17.2, R18.1, R19.1, U1.4 (FB), U3.2 (VDD), U4.16 (VCC)
- new net +5V: C1.2, J2.1 (Pin_1)
- new net +BATT: J24.1 (Pin_1), R1.1
- new net 5V: C4.1, C6.1, C8.2, D1.1 (K), J11.4 (Pin_4), U2.3 (VI)
- new net AD0: J1.7 (Pin_7)
- new net CS: U3.29 (IO5)
- new net DTR: Q1.2 (B1), Q1.4 (E2), U4.13 (~{DTR})
- new net EN: C5.2, Q1.6 (C1), R15.1, SW2.2, U3.3 (EN)
- new net GND: C1.1, C10.2, C11.2, C12.2, C13.1, C14.1, C15.2, C2.1, C3.2, C4.2, C5.1, C6.2, C7.1, C8.1, C9.2, D1.2 (A), D10.1 (K), D2.2 (A), D3.1 (K), D7.1 (K), D8.1 (K), D9.1 (K), J1.2 (Pin_2), J10.1 (Pin_1), J11.1 (Pin_1), J2.4 (Pin_4), J3.2 (Pin_2), J6.1 (Pin_1), R2.1, R8.1, SW2.1, SW3.1, U1.3 (GND), U1.5 (~{ON}/OFF), U1.6 (GND), U2.1 (GND), U3.1 (GND), U3.15 (GND), U3.38 (GND), U3.39 (GND), U4.1 (GND)
- new net GPIO0: Q1.3 (C2), R17.1, SW3.2, U3.25 (IOA0)
- new net GPIO12: R3.2, R8.2, U3.14 (IOA12)
- new net GPIO13: R4.1, U3.16 (IOA13)
- new net GPIO14: J2.2 (Pin_2), R5.1, U3.13 (IOA14)
- new net GPIO15: U3.23 (IOA15)
- new net GPIO16: R6.1, U3.27 (IO16)
- new net GPIO17: R7.1, U3.28 (IO17)
- new net GPIO1/TX: D5.1 (K), U3.35 (TXD0/IO1), U4.3 (RXD)
- new net GPIO2: R16.1, U3.24 (IOA2)
- new net GPIO25: U3.10 (IOA25)
- new net GPIO26: U3.11 (IOA26)
- new net GPIO27: J1.8 (Pin_8), U3.12 (IOA27)
- new net GPIO32: U3.8 (IOA32)
- new net GPIO33: U3.9 (IOA33)
- new net GPIO34: C2.2, R1.2, R2.2, U3.6 (IA34)
- new net GPIO35: U3.7 (IA35)
- new net GPIO36: U3.4 (IA36)
- new net GPIO39: U3.5 (IA39)
- new net GPIO3/RX: D6.1 (K), U3.34 (RXD0/IO3), U4.2 (TXD)
- new net GPIO4: U3.26 (IOA4)
- new net MISO: U3.31 (IO19)
- new net MOSI: U3.37 (IO23)
- new net RTS: Q1.1 (E1), Q1.5 (B2), U4.14 (~{RTS})
- new net SCK: U3.30 (IO18)
- new net SCL: J1.3 (Pin_3), R13.2, U3.36 (IO22)
- new net SDA: J1.4 (Pin_4), R14.1, U3.33 (IO21)
- new net VCC: C3.1, J9.1 (Pin_1), U1.1 (VIN)
- new net XCL: J1.6 (Pin_6)
- new net XDA: J1.5 (Pin_5)
- no-connect marks 0 -> 10
Other:
- note added: "3S LITHIUM BATTERY PACK"
- note added: "BATTERY LEVEL"
- note added: "BATTERY MANAGEMENT"
- note added: "COMMAND MICROCONTROLLER"
- note added: "DEBUGGING & PROGRAMMING"
- note added: "GYROSCOPE SENSOR"
- note added: "If CH340G is used"
- note added: "LED INDICATORS"
- note added: "MICROCONTROLLER COPROCESSOR"
- note added: "POWER SUPPLY"
- note added: "SYSTEM"
- note added: "ULTRASONIC SENSOR"

Commit message: update from work
Parts:
- added C16, C17, C18, C20, C21, C22, C23: 680uF_35V, Capacitor_SMD:CP_Elec_10x12.5, symbol PCM_SL_Capacitors:470uF_35V
- added C19, C25, C28: 100nF, Capacitor_SMD:C_0805_2012Metric_Pad1.18x1.45mm_HandSolder, symbol PCM_SL_Capacitors:104_Ceramic
- added C24: 470uF_16V, Capacitor_SMD:CP_Elec_10x12.5, symbol PCM_SL_Capacitors:470uF_35V
- added C26, C27: 220uF_16V, Capacitor_SMD:CP_Elec_10x12.5, symbol PCM_SL_Capacitors:470uF_35V
- added D11: 1N5824, Diode_SMD:D_SMA, symbol Diode:1N5822
- added J12: UART, symbol Connector:Screw_Terminal_01x04
- added J13: 12V IN, symbol Connector:Screw_Terminal_01x02
- added J14: MOTOR 4, symbol Connector:Screw_Terminal_01x06
- added J15: MOTOR 3, symbol Connector:Screw_Terminal_01x06
- added J16: MOTOR 2, symbol Connector:Screw_Terminal_01x06
- added J17: MOTOR 1, symbol Connector:Screw_Terminal_01x06
- added J4: I2C, symbol Connector:Screw_Terminal_01x04
- added L2: 33uH, Inductor_SMD:L_12x12mm_H6mm, symbol Device:L_Small
- added M1, M2, M3, M4: MOTOR, symbol Motor:Stepper_Motor_unipolar_6pin
- added U5: LM2596S-5V, Package_TO_SOT_SMD:TO-263-5_TabPin6, symbol Regulator_Switching:LM2596S-3.3
- C10: value 220uF_16V -> 470uF_16V; footprint Capacitor_SMD:CP_Elec_6.3x7.7 -> Capacitor_SMD:CP_Elec_10x12.5
- J10: value -5V -> OUT-
- J7: value -BATT -> 0V
- J8: value +BATT -> 12V6
- J9: value +5V -> OUT+
- R1: value 10k -> 68k
- R2: value 20k -> 18k
Connections:
- net +3.3V: now also C26.1, C28.2
- net +5V: now also C24.1, C25.2, C27.1, J12.4 (Pin_4), J4.4 (Pin_4), L2.2, U5.4 (FB)
- net GND: now also C16.2, C17.2, C18.2, C19.1, C20.2, C21.2, C22.2, C23.2, C24.2, C25.1, C26.2, C27.2, C28.1, D11.2 (A), J12.3 (Pin_3), J13.1 (Pin_1), J4.3 (Pin_3), U5.3 (GND), U5.5 (~{ON}/OFF), U5.6 (GND)
- net GPIO12: no longer R3.2, R8.2
- net GPIO14: no longer J2.2 (Pin_2)
- net GPIO16: now also J12.2 (Pin_2); no longer R6.1
- net GPIO17: now also J12.1 (Pin_1); no longer R7.1
- net GPIO26: now also R3.2, R8.2
- net GPIO27: now also J2.2 (Pin_2); no longer J1.8 (Pin_8)
- net GPIO35: now also J1.8 (Pin_8)
- net SCL: now also J4.2 (Pin_2)
- net SDA: now also J4.1 (Pin_1)
- net VCC: now also C16.1, C17.1, C18.1, C19.2, C20.1, C21.1, C22.1, C23.1, J13.2 (Pin_2), U5.1 (VIN)
- net 5V: no longer names the net of C4.1, C6.1, C8.2, D1.1 (K), J11.4 (Pin_4), U2.3 (VI)
- net MISO renamed GPIO19
- net GPIO19: now also R7.1
- net SCK renamed GPIO18
- net GPIO18: now also R6.1
- new net: J16.3V3 (Pin_2), M2.2
- new net: J16.GND (Pin_5), M2.5
- new net: J16.H1A (Pin_3), M2.3 (-)
- new net: J16.H1B (Pin_4), M2.4
- new net: J16.M+ (Pin_6), M2.6
- new net: J16.M- (Pin_1), M2.1
- new net: D11.1 (K), L2.1, U5.2 (OUT)
- new net: J14.M- (Pin_1), M4.1
- new net: J14.3V3 (Pin_2), M4.2
- new net: J14.H1A (Pin_3), M4.3 (-)
- new net: J14.H1B (Pin_4), M4.4
- new net: J14.GND (Pin_5), M4.5
- new net: J14.M+ (Pin_6), M4.6
- new net: J17.M- (Pin_1), M1.1
- new net: J17.3V3 (Pin_2), M1.2
- new net: J17.H1A (Pin_3), M1.3 (-)
- new net: J17.H1B (Pin_4), M1.4
- new net: J17.GND (Pin_5), M1.5
- new net: J17.M+ (Pin_6), M1.6
- new net: J15.M- (Pin_1), M3.1
- new net: J15.3V3 (Pin_2), M3.2
- new net: J15.H1A (Pin_3), M3.3 (-)
- new net: J15.H1B (Pin_4), M3.4
- new net: J15.GND (Pin_5), M3.5
- new net: J15.M+ (Pin_6), M3.6
- no-connect marks 10 -> 13
Other:
- note added: "COPROCESSOR 4-CHANNEL MOTOR DRIVER BOARD"
- moved on the sheet: BT1, BT2, BT3, BT4, BT5, BT6, C10, C13, C3, C5, C7, D2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

Commit message: update from work
Parts:
- added C1: 100nF, Capacitor_SMD:C_0805_2012Metric_Pad1.18x1.45mm_HandSolder, symbol PCM_SL_Capacitors:104_Ceramic
- added C2: 680uF_35V, Capacitor_SMD:CP_Elec_10x12.5, symbol PCM_SL_Capacitors:470uF_35V
- added C31: 470uF_16V, Capacitor_SMD:CP_Elec_10x12.5, symbol PCM_SL_Capacitors:470uF_35V
- added C32: 220uF_16V, Capacitor_SMD:CP_Elec_10x12.5, symbol PCM_SL_Capacitors:470uF_35V
- added J19: BMS, TerminalBlock_Phoenix:TerminalBlock_Phoenix_PT-1,5-2-5.0-H_1x02_P5.00mm_Horizontal, symbol Connector_Generic:Conn_01x02
- added J20: CHARGER, PCM_SparkFun-Connector:Barrel_Jack_PTH_Slot, symbol Connector_Generic:Conn_01x02
- added JP2, JP5, JP6: ~, Jumper:SolderJumper-2_P1.3mm_Open_Pad1.0x1.5mm, symbol SparkFun-Jumper:SolderJumper_2_Open
- added JP3, JP4: SolderJumper_3_Open, Jumper:SolderJumper-3_P1.3mm_Open_Pad1.0x1.5mm, symbol Jumper:SolderJumper_3_Open
- added M1: Motor_Servo, Connector_PinHeader_2.54mm:PinHeader_1x03_P2.54mm_Vertical, symbol Motor:Motor_Servo
- added R16: 10k, Resistor_SMD:R_0805_2012Metric, symbol PCM_SL_Resistors:10k
- added R17: 20k, Resistor_SMD:R_0805_2012Metric, symbol PCM_SL_Resistors:10k
- J12: renamed from J9; now left out of the parts list
- J13: renamed from J10; now left out of the parts list
- J14: renamed from J1; footprint (none) -> Connector_PinHeader_2.54mm:PinHeader_1x08_P2.54mm_Vertical
- J15: renamed from J12; footprint (none) -> Connector_PinHeader_2.00mm:PinHeader_1x04_P2.00mm_Vertical
- J16: renamed from J4; footprint (none) -> Connector_PinHeader_2.00mm:PinHeader_1x04_P2.00mm_Vertical
- J17: renamed from J13; footprint (none) -> TerminalBlock_Phoenix:TerminalBlock_Phoenix_PT-1,5-2-5.0-H_1x02_P5.00mm_Horizontal
- J3: renamed from J5; now left out of the parts list
- J4: renamed from J6; now left out of the parts list
- renumbered BT3 to BT1, BT4 to BT2, BT1 to BT3, BT2 to BT4, C23 to C10, C4 to C11, C16 to C12, C6 to C13, C5 to C14, C17 to C15, C7 to C16, C18 to C17, C8 to C18, C9 to C19, C19 to C20, C11 to C21, C12 to C22, C14 to C23, C10 to C24, C24 to C25, C15 to C26, C26 to C27, C27 to C28, C13 to C29, C2 to C3, C25 to C30, C28 to C4, C1 to C5, C3 to C6, C20 to C7, C21 to C8, C22 to C9, D7 to D1, D11 to D10, D6 to D11, D8 to D2, D9 to D3, D10 to D4, D1 to D5, D3 to D6, D4 to D7, D5 to D8, D2 to D9, J24 to J1, J16 to J10, J14 to J11, J11 to J18, J3 to J2, J7 to J5, J17 to J6, J15 to J7, J2 to J9, M3 to M2, M1 to M3, M2 to M5, R4 to R1, R14 to R10, R15 to R11, R16 to R12, R17 to R13, R18 to R14, R19 to R15, R5 to R2, R1 to R3, R2 to R4, R6 to R5, R7 to R6, R3 to R7, R13 to R9, SW2 to SW1, SW3 to SW2, U2 to U1, U1 to U2, U5 to U3, U3 to U4, U4 to U5
Connections:
- net +3.3V: now also C31.1, C32.1, JP3.3 (B), JP4.3 (B)
- net +5V: now also C1.2, C2.1, JP3.1 (A), JP4.1 (A), M1.2 (+); no longer J15.4 (Pin_4), J16.4 (Pin_4)
- net GND: now also J17.2 (Pin_2), C1.1, C2.2, C31.2, C32.2, J19.2 (Pin_2), J20.2 (Pin_2), M1.3 (-), R16.2; no longer J17.1 (Pin_1)
- net GPIO16: now also JP2.1 (A), R16.1, R17.2; no longer J15.2 (Pin_2)
- net GPIO25: now also M1.1 (PWM)
- net SCL: now also JP5.2 (B); no longer J16.2 (Pin_2)
- net SDA: now also JP6.2 (B); no longer J16.1 (Pin_1)
- net VCC: now also J17.1 (Pin_1), J19.1 (Pin_1), J20.1 (Pin_1); no longer J17.2 (Pin_2)
- net +: now reaches J18.2 (Pin_2), U5.5 (UD+)
- net -: now reaches J18.3 (Pin_3), U5.6 (UD-)
- new net: J15.2 (Pin_2), JP2.2 (B), R17.1
- new net: J16.1 (Pin_1), JP6.1 (A)
- new net: J16.2 (Pin_2), JP5.1 (A)
- new net A: J15.4 (Pin_4), JP4.2 (C)
- new net B: J16.4 (Pin_4), JP3.2 (C)
- no-connect marks 13 -> 12
Other:
- note added: "SERVO"
- moved on the sheet: C3, D1, D2, D3, D4, M2, M3, M4, M5, R1, R2, R3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

Commit message: update from home
Connections:
- net GPIO13: now also R6.1; no longer R1.1
- net GPIO14: now also R5.1; no longer R2.1
- net GPIO18: now also R1.1; no longer R5.1
- net GPIO19: now also R2.1; no longer R6.1
Changed lines of the file:
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@@
 	)
 	(label "GPIO19"
-		(at 132.08 231.14 270)
+		(at 113.03 231.14 270)
 		(effects
 			(font
@@
 	)
 	(label "GPIO18"
-		(at 121.92 231.14 270)
+		(at 104.14 231.14 270)
 		(effects
 			(font
@@
 	)
 	(label "GPIO14"
-		(at 113.03 231.14 270)
+		(at 121.92 231.14 270)
 		(effects
 			(font
@@
 	)
 	(label "GPIO13"
-		(at 104.14 231.14 270)
+		(at 132.08 231.14 270)
 		(effects
 			(font
