File: ESP32/Smart Robotic Car With PID control/hardware/Smart Robotic Car With PID control.kicad_pcb (KiCad board)
At the start: 2 copper layers, 275 x 148 mm, 87 parts, among them J1 BSENS, J14 MPU6050, J15 UART, J16 I2C, J17 12V IN, J18 USB_C Conn, J19 BMS, J20 CHARGER, J9 Ultra Sonic, M1 Motor_Servo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

Commit message: update from home
Parts:
- added G***: LOGO, logo:CULogo, F.Cu at (91.5, 146.5)
Connections:
- R1 pad 1: /GPIO13 -> /GPIO18
- R2 pad 1: /GPIO14 -> /GPIO19
- R5 pad 1: /GPIO18 -> /GPIO14
- R6 pad 1: /GPIO19 -> /GPIO13
Routing:
- net /GPIO18: track 0.00 -> 246.3 mm, vias 0 -> 4
- net /GPIO19: track 0.00 -> 239.5 mm, vias 0 -> 2
- net /GPIO2: track 0.00 -> 221.3 mm, vias 0 -> 2
- net /GPIO14: track 0.00 -> 216.6 mm, vias 0 -> 2
- net /GPIO13: track 0.00 -> 209.4 mm, vias 0 -> 4
- net /GPIO17: track 0.00 -> 206.9 mm, vias 0 -> 2
- net +3.3V: track 133.3 -> 340.1 mm, vias 0 -> 2
- net /B: track 0.00 -> 189.5 mm, vias 0 -> 3
- net /A: track 0.00 -> 186.4 mm, vias 0 -> 3
- net /GPIO3/RX: track 0.00 -> 177.0 mm, vias 0 -> 4
- net Net-(J16-Pin_2): track 0.00 -> 171.2 mm, vias 0 -> 2
- net Net-(J16-Pin_1): track 0.00 -> 171.1 mm, vias 0 -> 3
- net Net-(J15-Pin_2): track 4.50 -> 171.7 mm, vias 0 -> 4
- net /GPIO1/TX: track 0.00 -> 166.5 mm, vias 0 -> 4
- net /GPIO34: track 8.69 -> 135.2 mm, vias 0 -> 4
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Other:
- outline, holes or cut-outs redrawn
- board text added: "+12"
- board text added: "+5V"
- board text added: "D+"
- board text added: "D-"
- board text added: "ECHO"
- board text added: "RX"
- board text added: "SIG"
- board text added: "TRIG"
- board text added: "TX"
- board text added: "VCC"

Commit message: Reference materials updated
Parts:
- moved R12 4.77 mm to (339.7, 136.5)
- moved R1 4.77 mm to (339.7, 112.2)
- moved R6 4.77 mm to (339.7, 130.2)
- moved R5 4.77 mm to (339.7, 124.2)
- moved R2 4.77 mm to (339.7, 118.2)
- moved C20 2.70 mm to (333.1, 160.4)
- moved R7 1.82 mm to (153.2, 169.0)
Routing:
- net Net-(D6-A): track 2.52 -> 7.35 mm
- net Net-(D1-A): track 2.52 -> 7.34 mm
- net Net-(D4-A): track 2.52 -> 7.34 mm
- net Net-(D3-A): track 2.52 -> 7.31 mm
- net Net-(D2-A): track 2.52 -> 7.31 mm
- net /GPIO13: track 209.4 -> 204.6 mm
- net /GPIO2: track 221.3 -> 216.6 mm
- net /A: track 186.4 -> 190.1 mm
- net /GPIO14: track 216.6 -> 214.1 mm
- net /GPIO26: track 45.6 -> 47.4 mm
- net Net-(J9-Pin_3): track 4.45 -> 6.27 mm
- net /GPIO18: track 246.3 -> 245.0 mm
- net /B: track 189.5 -> 188.7 mm
- net GND: vias 169 -> 180
Other:
- outline, holes or cut-outs redrawn
- board text added: "+12.6V"
- board text added: "100%"
- board text added: "25%"
- board text added: "50%"
- board text added: "75%"
- board text added: "BMS_IN"
- board text added: "CHARGER"
- board text added: "COPROCESSOR 4 MOTOR DRIVER WITH ENCODER"
- board text added: "GYROSCOPE"
- board text added: "LITHIUM ION BATTERY"
- board text added: "MICROCONTROLLER"
- board text added: "P_ON"
- board text added: "SERVO"
- board text added: "SERVO MOTOR SLOT"
- board text added: "SONIC"
- board text added: "USB"
