File: ESP32/Predictive Maintenance System for Industrial Motor/hardware/Predictive Maintenance System for Industrial Motor.kicad_sch (KiCad schematic)
At the start: 80 parts, among them J1 220VAC, J11 LOAD, J16 SD MODULE, J17 MPU6050, J3 AM2301A, J4 OLED SCREEN, J5 CURRENT SENSOR, J7 USB_C Conn, K1 FINDER-36.11, Q3 UMH3N, SW1 RotaryEncoder, SW2 RESET, SW3 FLASH, T3 2220-12V, U1 AMS1117-3.3, U3 LM2596S-3.3V, U4 LM2596S-3.3V, U5 CH340C, U6 ESP32-S3-WROOM-1U-N16R8, Y1 12MHz

Commit message: Update from work
Parts:
- removed T3: 2220-12V, symbol Device:Transformer_1P_1S
- added C25: 4.7uF/16V, Capacitor_Tantalum_SMD:CP_EIA-3528-21_Kemet-B_HandSolder, symbol PCM_SL_Capacitors:4.7uF_16V
- added J9: 12VAC, TerminalBlock_Phoenix:TerminalBlock_Phoenix_MKDS-1,5-2_1x02_P5.00mm_Horizontal, symbol Connector_Generic:Conn_01x02
- D1: footprint PCM_Diode_THT_AKL:D_DO-41_SOD81_P7.62mm_Horizontal -> Diode_SMD:D_SMA
- J1: renamed from J3; value AM2301A -> DS18B20
- J4: renamed from J11; footprint TerminalBlock_Phoenix:TerminalBlock_Phoenix_PT-1,5-2-3.5-H_1x02_P3.50mm_Horizontal -> TerminalBlock_Phoenix:TerminalBlock_Phoenix_MKDS-1,5-2_1x02_P5.00mm_Horizontal
- J5: renamed from J1; footprint TerminalBlock_Phoenix:TerminalBlock_Phoenix_PT-1,5-2-3.5-H_1x02_P3.50mm_Horizontal -> TerminalBlock_Phoenix:TerminalBlock_Phoenix_MKDS-1,5-2_1x02_P5.00mm_Horizontal
- U2: renamed from U6; footprint ESP32-S3-WROOM-1U-N16R8:XCVR_ESP32-S3-WROOM-1U-N16R8 -> footprints:ESP32-S3-WROOM-1U-N16R8
- U4: value LM2596S-3.3V -> LM2596S-5V
- renumbered C9 to C10, C10 to C11, C11 to C12, C12 to C13, C42 to C14, C13 to C15, C14 to C16, C15 to C17, C16 to C18, C17 to C19, C18 to C20, C19 to C21, C20 to C22, C21 to C23, C22 to C24, C5 to C3, C3 to C5, C24 to C6, C41 to C7, C7 to C8, C8 to C9, D5 to D10, D6 to D11, D7 to D12, D8 to D13, D32 to D2, D33 to D3, D3 to D4, D34 to D5, D35 to D6, D2 to D7, D31 to D8, D4 to D9, DZ2 to DZ1, J5 to J2, J4 to J3, J17 to J6, J16 to J7, J7 to J8, OC3 to OC1, OC1 to OC2, Q3 to Q1, R5 to R1, R25 to R10, R26 to R11, R10 to R12, R9 to R13, R11 to R14, R12 to R15, R13 to R16, R6 to R2, R7 to R3, R1 to R4, R15 to R5, R14 to R6, R2 to R7, R3 to R8, R4 to R9
Connections:
- net +3.3V: no longer C5.2
- net +5V: now also C5.2
- net GND: now also U2.41 (GND); no longer OC1.3, U2.41_1 (GND), U2.41_2 (GND), U2.41_3 (GND), U2.41_4 (GND), U2.41_5 (GND), U2.41_6 (GND), U2.41_7 (GND), U2.41_8 (GND), U2.41_9 (GND)
- net GNDA: now also OC1.3
- net LIVE: now also J5.1 (Pin_1); no longer J5.2 (Pin_2)
- net NEUTRAL: now also J4.1 (Pin_1), J5.2 (Pin_2); no longer J4.2 (Pin_2), J5.1 (Pin_1)
- net VCC2: now also C25.1
- net at K1.14: now also J4.2 (Pin_2); no longer J4.1 (Pin_1)
- net at D8.2: now also J9.1 (Pin_1)
- net at D8.3: now also J9.2 (Pin_2)
- net at D1.2 (A), K1.A2, OC1.4: now also C25.2
Other:
- moved on the sheet: D1, J4, J5, R1
