File: ESP32/Predictive Maintenance System for Industrial Motor/hardware/Predictive Maintenance System for Industrial Motor.kicad_pcb (KiCad board)
At the start: 2 copper layers, 108.8 x 83.6 mm, 86 parts, among them J1 DS18B20, J2 CURRENT SENSOR, J3 OLED SCREEN, J4 LOAD, J5 220VAC, J6 MPU6050, J7 SD MODULE, J8 USB_C Conn, J9 12VAC, K1 FINDER-36.11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

Commit message: Update from work
Parts:
- added G***: LOGO, logo:CULogo, B.Cu at (145.2, 75.6)
- moved R3 0.75 mm to (95.6, 98.7)
- moved J6 0.39 mm to (86.3, 95.8)
- moved C24 0.39 mm to (133.1, 88.7)
Routing:
- net GNDA: track 34.9 -> 37.8 mm
- net Net-(JP1-A): track 34.2 -> 35.1 mm
- net +3.3V: track 277.5 -> 278.4 mm
- net +5V: track 129.5 -> 128.8 mm
Other:
- outline, holes or cut-outs redrawn
- board text added: "+5V"
- board text added: "A"
- board text added: "B"
- board text added: "BUZZER"
- board text added: "D+"
- board text added: "D-"
- board text added: "ENCODER"
- board text added: "INT1"
- board text added: "INT2"
- board text added: "LIVE"
- board text added: "MICROCONTROLLER"
- board text added: "N"
- board text added: "SCL"
- board text added: "SCREEN"
- board text added: "SD0"
- board text added: "SDA"
- board text added: "SENSOR 1"
- board text added: "SENSOR 2"
- board text added: "SENSOR 3"
- board text added: "SIG"
- board text added: "SW"
