File: ESP32/Solar Powered Egg Incubator/Solar Powered Egg Incubator.kicad_sch (KiCad schematic)
At the start: 61 parts, among them J1 BMS, J10 SPINNER, J11 HUMIDIFIER, J12 SCREEN, J13 MAIN, J2 GLCD, J3 ULTRASONIC, J4 RTC, J5 AHT20, J6 PROG, J7 Buzzer, J8 LEVELS, J9 HEATER, K1 RELAY, K2 RELAY, K3 RELAY, SW1 RotaryEncoder_Switch, SW2 RESET, U1 LM2596S-5.0, U2 LM2596S-3.3, U3 ESP32-WROOM-32

Commit message: sync updates
Parts:
- removed C1, C2, C5, C6: 220uF/35V, Capacitor_THT:CP_Radial_D8.0mm_P3.80mm, symbol Device:C_Polarized_Small
- removed C10, C11, C9: 10uF, Capacitor_THT:CP_Radial_D5.0mm_P2.50mm, symbol Device:C_Polarized_Small
- removed C3, C4, C7, C8: 0.1uF, Capacitor_THT:C_Disc_D7.0mm_W2.5mm_P5.00mm, symbol Device:C_Small
- removed D1, D2: SS34, Diode_SMD:D_SMA, symbol Diode:SS34
- removed D5, D6, D7: 1N4007, Diode_THT:D_DO-41_SOD81_P10.16mm_Horizontal, symbol Diode:1N4007
- removed J10: SPINNER, TerminalBlock_Phoenix:TerminalBlock_Phoenix_PT-1,5-2-3.5-H_1x02_P3.50mm_Horizontal, symbol PCM_SL_Screw_Terminal:Screw_Terminal_2_P3.50mm
- removed J11: HUMIDIFIER, TerminalBlock_Phoenix:TerminalBlock_Phoenix_PT-1,5-2-3.5-H_1x02_P3.50mm_Horizontal, symbol PCM_SL_Screw_Terminal:Screw_Terminal_2_P3.50mm
- removed J12: SCREEN, Connector_PinHeader_2.54mm:PinHeader_1x12_P2.54mm_Vertical, symbol Connector:Screw_Terminal_01x12
- removed J13: MAIN, Connector_PinHeader_2.54mm:PinHeader_1x12_P2.54mm_Vertical, symbol Connector:Screw_Terminal_01x12
- removed J2: GLCD, Connector_PinSocket_2.54mm:PinSocket_1x20_P2.54mm_Vertical, symbol Connector:Screw_Terminal_01x20
- removed J3: ULTRASONIC, TerminalBlock_Phoenix:TerminalBlock_Phoenix_PT-1,5-4-3.5-H_1x04_P3.50mm_Horizontal, symbol PCM_SL_Screw_Terminal:Screw_Terminal_4_P3.50mm
- removed J6: PROG, Connector_PinHeader_2.54mm:PinHeader_2x03_P2.54mm_Vertical, symbol Connector:Screw_Terminal_01x06
- removed J7: Buzzer, TerminalBlock_Phoenix:TerminalBlock_Phoenix_PT-1,5-2-3.5-H_1x02_P3.50mm_Horizontal, symbol PCM_SL_Screw_Terminal:Screw_Terminal_2_P3.50mm
- removed J9: HEATER, TerminalBlock_Phoenix:TerminalBlock_Phoenix_PT-1,5-2-5.0-H_1x02_P5.00mm_Horizontal, symbol PCM_SL_Screw_Terminal:Screw_Terminal_2_P3.50mm
- removed K1, K2, K3: RELAY, Relay_THT:Relay_SPDT_Finder_36.11, symbol Relay:FINDER-36.11
- removed OC1, OC2, OC3, OC4: PC817, PCM_Package_DIP_AKL:DIP-4_W7.62mm_LongPads, symbol PCM_Optocoupler_AKL:PC817
- removed R12, R13, R14, R15: 150R, Resistor_THT:R_Axial_DIN0207_L6.3mm_D2.5mm_P10.16mm_Horizontal, symbol PCM_SL_Resistors:10k
- removed R3, R6, R7: 10k, Resistor_THT:R_Axial_DIN0207_L6.3mm_D2.5mm_P10.16mm_Horizontal, symbol PCM_SL_Resistors:10k
- removed SW1: RotaryEncoder_Switch, Rotary_Encoder:RotaryEncoder_Alps_EC11E-Switch_Vertical_H20mm, symbol Device:RotaryEncoder_Switch
- removed SW2: RESET, Button_Switch_THT:SW_PUSH_6mm_H5mm, symbol Switch:SW_Push
- removed U2: LM2596S-3.3, Package_TO_SOT_SMD:TO-263-5_TabPin3, symbol Regulator_Switching:LM2596S-3.3
- removed U3: ESP32-WROOM-32, RF_Module:ESP32-WROOM-32, symbol RF_Module:ESP32-WROOM-32
- removed VR1: 10k, PCM_Potentiometer_THT_AKL:Potentiometer_Bourns_3296W_Vertical, symbol 3296W-OT1-103LF:3296W-OT1-103LF
- added BZ6: Buzzer, Buzzer_Beeper:Buzzer_15x7.5RM7.6, symbol Device:Buzzer
- added C1, C22, C30, C5, C55, C59, C60, C8, C9: 100nF, Capacitor_SMD:C_0805_2012Metric_Pad1.18x1.45mm_HandSolder, symbol PCM_SL_Capacitors:104_Ceramic
- added C10, C4: 220uF_16V, Capacitor_SMD:CP_Elec_6.3x7.7, symbol PCM_SL_Capacitors:470uF_35V
- added C18, C24: 4.7uF/16V, Capacitor_Tantalum_SMD:CP_EIA-3528-21_Kemet-B_HandSolder, symbol PCM_SL_Capacitors:4.7uF_16V
- added C19: 470nF, Capacitor_SMD:C_0805_2012Metric_Pad1.18x1.45mm_HandSolder, symbol PCM_SL_Capacitors:104_Ceramic
- added C2, C3, C6, C7: 680uF_35V, Capacitor_SMD:CP_Elec_10x12.5, symbol PCM_SL_Capacitors:470uF_35V
- added C20: 10uF_16V, Capacitor_THT:CP_Radial_D5.0mm_P2.00mm, symbol PCM_SL_Capacitors:10uF_16V
- added C23, C28: 100nF, Capacitor_SMD:C_0805_2012Metric_Pad1.18x1.45mm_HandSolder, symbol Device:C_Small
- added C25, C26: 22pF, Capacitor_SMD:C_0805_2012Metric_Pad1.18x1.45mm_HandSolder, symbol Device:C_Small
- added C56, C57, C58: 10uF, Capacitor_Tantalum_SMD:CP_EIA-3528-21_Kemet-B_HandSolder, symbol Device:C_Polarized_Small
- added D1, D2: 1N5824, Diode_SMD:D_SMA, symbol Diode:1N5822
- added D11, D8: Red, LED_THT:LED_D3.0mm, symbol SparkFun-LED:LED_Red_0603
- added D12: Green, LED_THT:LED_D3.0mm, symbol SparkFun-LED:LED_Red_0603
- added D14, D9: 1N5819, Diode_SMD:D_SMA, symbol Diode:1N5819
- added D23, D24, D25: 1N4007, Diode_SMD:D_SMA, symbol Diode:1N4007
- added J2: SPINNER, TerminalBlock_Phoenix:TerminalBlock_Phoenix_MKDS-1,5-3_1x03_P5.00mm_Horizontal, symbol PCM_SL_Screw_Terminal:Screw_Terminal_3_P3.50mm
- added J23: USB_C Conn, Connector_PinHeader_2.54mm:PinHeader_1x04_P2.54mm_Vertical, symbol Connector:Screw_Terminal_01x04
- added J3: BMS, TerminalBlock_Phoenix:TerminalBlock_Phoenix_PT-1,5-2-5.0-H_1x02_P5.00mm_Horizontal, symbol PCM_SL_Screw_Terminal:Screw_Terminal_2_P3.50mm
- added J42: Ultra Sonic, Connector_PinSocket_2.54mm:PinSocket_1x04_P2.54mm_Vertical, symbol Connector:Screw_Terminal_01x04
- added J47: SCREEN, Connector_PinHeader_2.54mm:PinHeader_1x12_P2.54mm_Vertical, symbol Connector:Screw_Terminal_01x12
- added J6: HUMIDIFIER, TerminalBlock_Phoenix:TerminalBlock_Phoenix_MKDS-1,5-3_1x03_P5.00mm_Horizontal, symbol PCM_SL_Screw_Terminal:Screw_Terminal_3_P3.50mm
- added J7: HEATER, TerminalBlock_Phoenix:TerminalBlock_Phoenix_MKDS-1,5-3_1x03_P5.00mm_Horizontal, symbol PCM_SL_Screw_Terminal:Screw_Terminal_3_P3.50mm
- added JP1: SolderJumper_3_Open, Jumper:SolderJumper-3_P1.3mm_Open_Pad1.0x1.5mm, symbol Jumper:SolderJumper_3_Open
- added JP2, JP3, JP4, JP5: ~, Jumper:SolderJumper-2_P1.3mm_Open_Pad1.0x1.5mm, symbol SparkFun-Jumper:SolderJumper_2_Open
- added K4, K5, K6: RELAY, Relay_THT:Relay_SPDT_Finder_36.11, symbol Relay:FINDER-36.11
- added OC1, OC10, OC11, OC8, OC9: PC817XI, PCM_Package_DIP_AKL:SMDIP-4_W9.53mm, symbol PCM_Optocoupler_AKL:PC817XI
- added OC13, OC14: PC817, PCM_Package_DIP_AKL:SMDIP-4_W9.53mm, symbol PCM_Optocoupler_AKL:PC817XI
- added Q2: UMH3N, Package_TO_SOT_SMD:SOT-363_SC-70-6, symbol Transistor_BJT:UMH3N
- added Q9: TIP41, Package_TO_SOT_THT:TO-220-3_Vertical, symbol PCM_Transistor_BJT_AKL:TIP41
- added R26, R28, R34, R35, R48, R49, R50, R51: 10k, Resistor_SMD:R_0805_2012Metric, symbol PCM_SL_Resistors:10k
- added R27, R29, R30: 330R, Resistor_SMD:R_0805_2012Metric, symbol PCM_SL_Resistors:1M
- added R46: 1k, Resistor_SMD:R_0805_2012Metric, symbol PCM_SL_Resistors:10k
- added R47: 2k, Resistor_SMD:R_0805_2012Metric, symbol PCM_SL_Resistors:10k
- added R53, R54: 150R, Resistor_SMD:R_0805_2012Metric, symbol PCM_SL_Resistors:10k
- added RV2: 10K, Potentiometer_THT:Potentiometer_Bourns_3296W_Vertical, symbol Device:R_Potentiometer_Small
- added SW4: RESET, Button_Switch_SMD:SW_SPST_CK_KXT3, symbol PCM_SL_Devices:Push_Button
- added SW5: FLASH, Button_Switch_SMD:SW_SPST_CK_KXT3, symbol PCM_SL_Devices:Push_Button
- added SW6: RotaryEncoder, Connector_PinHeader_2.54mm:PinHeader_1x06_P2.54mm_Vertical, symbol Device:RotaryEncoder_Switch_MP
- added U3: LM2596S-5V, Package_TO_SOT_SMD:TO-263-5_TabPin6, symbol Regulator_Switching:LM2596S-3.3
- added U5: AMS1117-3.3, Package_TO_SOT_SMD:SOT-223-3_TabPin2, symbol Regulator_Linear:AMS1117-3.3
- added U7: ESP32-WROOM, RF_Module:ESP32-WROOM-32, symbol SparkFun-RF:ESP32-WROOM
- added U8: CH340C, Package_SO:SOIC-16_3.9x9.9mm_P1.27mm, symbol Interface_USB:CH340C
- added Y2: 12MHz, Crystal:Crystal_HC49-4H_Vertical, symbol PCM_SL_Devices:Crystal_16MHz
- D3, D4: footprint Diode_THT:D_DO-41_SOD81_P10.16mm_Horizontal -> Diode_SMD:D_SOD-123
- J1: value BMS -> FAN
- J5: footprint TerminalBlock_Phoenix:TerminalBlock_Phoenix_PT-1,5-4-3.5-H_1x04_P3.50mm_Horizontal -> Connector_PinHeader_2.54mm:PinHeader_1x04_P2.54mm_Vertical
- J8: footprint TerminalBlock_Phoenix:TerminalBlock_Phoenix_PT-1,5-3-3.5-H_1x03_P3.50mm_Horizontal -> Connector_PinHeader_2.54mm:PinHeader_1x03_P2.54mm_Vertical
- L1, L2: value 47uH -> 33uH; footprint Inductor_THT:L_Axial_L7.0mm_D3.3mm_P12.70mm_Horizontal_Fastron_MICC -> Inductor_SMD:L_12x12mm_H6mm
- R1, R10, R11, R8, R9: footprint Resistor_THT:R_Axial_DIN0207_L6.3mm_D2.5mm_P10.16mm_Horizontal -> Resistor_SMD:R_0805_2012Metric
- R2: value 10k -> 47k; footprint Resistor_THT:R_Axial_DIN0207_L6.3mm_D2.5mm_P10.16mm_Horizontal -> Resistor_SMD:R_0805_2012Metric
- R4: value 1k -> 10k; footprint Resistor_THT:R_Axial_DIN0207_L6.3mm_D2.5mm_P10.16mm_Horizontal -> Resistor_SMD:R_0805_2012Metric
- R5: value 2k -> 10k; footprint Resistor_THT:R_Axial_DIN0207_L6.3mm_D2.5mm_P10.16mm_Horizontal -> Resistor_SMD:R_0805_2012Metric
- U1: value LM2596S-5.0 -> LM2596S-3.3V; footprint Package_TO_SOT_SMD:TO-263-5_TabPin3 -> Package_TO_SOT_SMD:TO-263-5_TabPin6
Connections:
- net +3.3V: now also L1.2, R4.1, R5.2, U1.4 (FB), C1.2, C10.1, C22.2, C30.1, C59.2, C60.2, D9.1 (K), JP2.2 (B), OC14.4, R26.2, R28.2, R29.1, R30.1, R34.2, R35.1, U7.2 (VDD), U8.16 (VCC); no longer L2.2
- net +5V: now also L2.2, BZ6.1 (+), C4.1, C5.2, C55.2, J42.1 (Pin_1), OC13.4, RV2.1, U3.4 (FB); no longer L1.2, U1.4 (FB)
- net BATT_LEVEL: now also C8.1, U7.6 (IA34)
- net BUZZER: now also R51.1, U7.26 (IOA4)
- net ECHO: now also R46.2, R47.2, U7.11 (IOA26); no longer R4.1, R5.2
- net EN: now also C19.2, Q2.6 (C1), R26.1, SW4.2, U7.3 (EN)
- net ENCODER_A: now also J47.8 (Pin_8), R35.2, SW6.A, U7.8 (IOA32)
- net ENCODER_B: now also J47.9 (Pin_9), R34.1, SW6.B, U7.9 (IOA33)
- net GND: now also D3.2 (A), D4.2 (A), J8.2, R10.1, R9.1, U1.6 (GND), C1.1, C10.2, C18.2, C19.1, C2.2, C20.2, C22.1, C23.1, C24.2, C25.2, C26.2, C28.1, C3.2, C30.2, C4.2, C5.1, C55.1, C59.1, C6.2, C60.1, C7.2, C8.2, C9.1, D1.2 (A), D14.2 (A), D2.2 (A), D8.1 (K), J2.3, J23.1 (Pin_1), J3.2, J42.4 (Pin_4), J47.1 (Pin_1), J47.10 (Pin_10), J47.11 (Pin_11), J6.3, J7.3, OC1.2, OC1.3, OC10.2, OC10.3, OC11.2, OC11.3, OC13.2, OC14.2, OC8.2, OC8.3, OC9.2, OC9.3, Q9.3 (E), R47.1, RV2.3, SW4.1, SW5.1, SW6.C, SW6.MP, SW6.S2, U3.3 (GND), U3.5 (~{ON}/OFF), U3.6 (GND), U5.1 (GND), U7.1 (GND), U7.15 (GND), U7.38 (GND), U7.39 (GND), U8.1 (GND); no longer J1.2, R5.1
- net GPIO0: now also Q2.3 (C2), R28.1, SW5.2, U7.25 (IOA0)
- net HEATER: now also R48.1, U7.27 (IO16)
- net HUMIDIFIER: now also R50.1, U7.30 (IO18)
- net SCL: now also R4.2, U7.36 (IO22)
- net SDA: now also R5.1, U7.33 (IO21)
- net SOLAR_LEVEL: now also C9.2, U7.7 (IA35)
- net SPINNER: now also R49.1, U7.28 (IO17)
- net TRIG: now also J42.2 (Pin_2), U7.12 (IOA27)
- net at L1.1, U1.2 (OUT): now also D2.1 (K)
- net at L2.1: now also D1.1 (K), U3.2 (OUT)
- net +3.3VA: no longer names the net of R1.2
- net +3.3VA: now also OC1.1; no longer R2.2
- net BMS_OUTPUT renamed VCC
- net VCC: now also R2.2, C2.1, C3.1, C56.1, C57.1, C58.1, C6.1, C7.1, D23.1 (K), D24.1 (K), D25.1 (K), J3.1, JP3.2 (B), JP4.2 (B), JP5.2 (B), K4.A2, K5.A2, K6.A2, U3.1 (VIN)
- net ENCODER_AA: no longer names the net of R2.1
- net ENCODER_AA: now also OC1.4, Q9.1 (B)
- net ENCODER_BA: no longer names the net of R1.1
- net ENCODER_BA: now also JP1.2 (C)
- new net: D11.2 (A), R29.2
- new net: J47.12 (Pin_12), RV2.2
- new net: OC9.1, R49.2
- new net: C57.2, D24.2 (A), K5.A1, OC9.4
- new net: J1.2, Q9.2 (C)
- new net: OC13.1, R53.1
- new net: J6.1, K4.14
- new net: C56.2, D23.2 (A), K4.A1, OC10.4
- new net: OC14.1, R54.1
- new net: J47.2 (Pin_2), OC14.3
- new net: C18.1, C20.1, C23.2, D14.1 (K), J23.4 (Pin_4), U5.3 (VI)
- new net: D8.2 (A), R27.2
- new net: C24.1, D9.2 (A), U5.2 (VO)
- new net: J47.3 (Pin_3), OC13.3
- new net: OC10.1, R50.2
- new net: C58.2, D25.2 (A), K6.A1, OC8.4
- new net: OC8.1, R48.2
- new net: D12.2 (A), R30.2
- new net: J2.1, K5.14
- new net: J7.1, K6.14
- new net: C28.2, JP2.1 (A), U8.4 (V3)
- new net: C25.1, U8.7 (Xi), Y2.2
- new net: C26.1, U8.8 (Xo), Y2.1
- new net: OC11.1, R51.2
- new net: BZ6.2 (-), OC11.4
- new net: J42.3 (Pin_3), R46.1
- new net +: J23.2 (Pin_2), U8.5 (UD+)
- new net -: J23.3 (Pin_3), U8.6 (UD-)
- new net A: J7.2, JP5.1 (A), K6.11
- new net B: J2.2, JP3.1 (A), K5.11
- new net C: J6.2, JP4.1 (A), K4.11
- new net DTR: Q2.2 (B1), Q2.4 (E2), U8.13 (~{DTR})
- new net ENCODER_SW: J47.7 (Pin_7), SW6.S1, U7.10 (IOA25)
- new net GPIO12: JP1.1 (A), U7.14 (IOA12)
- new net GPIO13/CS: J47.4 (Pin_4), U7.16 (IOA13)
- new net GPIO14/CLK: J47.6 (Pin_6), U7.13 (IOA14)
- new net GPIO15: R54.2, U7.23 (IOA15)
- new net GPIO19: R53.2, U7.31 (IO19)
- new net GPIO1/TX: D11.1 (K), U7.35 (TXD0/IO1), U8.3 (RXD)
- new net GPIO2: R27.1, U7.24 (IOA2)
- new net GPIO23/MOSI: J47.5 (Pin_5), U7.37 (IO23)
- new net GPIO36: U7.4 (IA36)
- new net GPIO39: U7.5 (IA39)
- new net GPIO3/RX: D12.1 (K), U7.34 (RXD0/IO3), U8.2 (TXD)
- new net GPIO5: JP1.3 (B), U7.29 (IO5)
- new net RTS: Q2.1 (E1), Q2.5 (B2), U8.14 (~{RTS})
- no-connect marks 20 -> 5
Other:
- note added: "BUZZER"
- note added: "CONTROL & COMMAND"
- note added: "DEBUGGING & PROGRAMMING"
- note added: "FAN"
- note added: "HEATER"
- note added: "HUMIDIFIER"
- note added: "If CH340G is used"
- note added: "POWER SUPPLY"
- note added: "REAL TIME CLOCK"
- note added: "SOLAR & BATTERY VOLTAGE LEVEL"
- note added: "SPINNER"
- note added: "TEMPERATURE & HUMIDITY SENSOR"
- note added: "ULTRASONIC SENSOR"
- note added: "USER INPUT & SCREEN"
- note removed: "ESP32-VROOM"
- moved on the sheet: D3, D4, J4, J5, J8, R10, R11, R8, R9
