File: ESP32/Solar Powered Egg Incubator/hardware/Solar Powered Egg Incubator.kicad_pcb (KiCad board)
At the start: 2 copper layers, 100 x 90.1 mm, 105 parts, among them J1 FAN, J2 SPINNER, J23 USB_C Conn, J3 BMS, J4 RTC, J42 Ultra Sonic, J47 SCREEN, J5 AHT20, J6 HUMIDIFIER, J7 HEATER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

Commit message: sync updates
Routing:
- net /TRIG: track 7.13 -> 90.9 mm, vias 1 -> 5
- net /SOLAR_LEVEL: track 34.1 -> 104.4 mm, vias 4 -> 5
- net /BATT_LEVEL: track 31.7 -> 98.6 mm, vias 2 -> 4
- net /GPIO15: track 0.00 -> 41.5 mm, vias 0 -> 4
- net VCC: track 230.9 -> 232.6 mm, vias 4 -> 45
- net /ECHO: track 98.7 -> 99.4 mm
- net GND: vias 14 -> 115
- added copper zone on B.Cu, net /A
- added copper zone on F.Cu, net /A
- added copper zone on B.Cu, net /B
- added copper zone on F.Cu, net /B
- added copper zone on B.Cu, net /C
- added copper zone on F.Cu, net /C
- added copper zone on B.Cu, net Net-(J2-Pad1)
- added copper zone on F.Cu, net Net-(J2-Pad1)
- added copper zone on B.Cu, net Net-(J6-Pad1)
- added copper zone on F.Cu, net Net-(J6-Pad1)
- added copper zone on B.Cu, net Net-(J7-Pad1)
- added copper zone on F.Cu, net Net-(J7-Pad1)
- added copper zone on B.Cu, net VCC
- added copper zone on F.Cu, net VCC
Other:
- outline, holes or cut-outs redrawn
- board text added: "+3V3"
- board text added: "+5V"
- board text added: "CLK"
- board text added: "CONST"
- board text added: "CS"
- board text added: "D+"
- board text added: "D-"
- board text added: "ECHO"
- board text added: "ENA"
- board text added: "ENB"
- board text added: "ENSW"
- board text added: "GND"
- board text added: "MOSI"
- board text added: "SCL"
- board text added: "SDA"
- board text added: "SIG"
- board text added: "TRIG"
