File: ESP32/NFC Card Payment System/hardware/NFC Card Payment System.kicad_sch (KiCad schematic)
At the start: 65 parts, among them J1 RTC, J10 -UPS, J11 V_OUT, J12 +BATT, J13 BUTTONS, J14 AS608, J15 SD MODULE, J16 -BATT, J17 SW_C, J18 SW_NO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

Commit message: sync updates
Parts:
- removed C10: 104, Capacitor_SMD:C_0805_2012Metric, symbol Device:C_Small
- removed J14: AS608, Connector_PinHeader_2.54mm:PinHeader_1x06_P2.54mm_Vertical, symbol Connector:Screw_Terminal_01x06
- U3: value RC522 -> PN532
Connections:
- no-connect marks 25 -> 23
Other:
- note removed: "SENSOR"
- moved on the sheet: 3.3V2, 3.3V5, 5V1, BT1, BT2, BZ1, C1, C11, C2, C3, C4, C5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
